File: ozprey_pcb/ozprey.kicad_pcb (KiCad board)
At the start: 2 copper layers, 263.5 x 99.3 mm, 95 parts, among them SW1 CPG135001S30, SW10 CPG135001S30, SW11 CPG135001S30, SW12 CPG135001S30, SW13 CPG135001S30, SW14 CPG135001S30, SW15 CPG135001S30, SW16 CPG135001S30, SW17 CPG135001S30, SW18 CPG135001S30, SW19 CPG135001S30, SW2 CPG135001S30, SW20 CPG135001S30, SW21 CPG135001S30, SW22 CPG135001S30, SW23 CPG135001S30, SW24 CPG135001S30, SW25 CPG135001S30, SW26 CPG135001S30, SW27 CPG135001S30, SW28 CPG135001S30, SW29 CPG135001S30, SW3 CPG135001S30, SW30 CPG135001S30, SW31 CPG135001S30, SW32 CPG135001S30, SW33 CPG135001S30, SW34 CPG135001S30, SW35 CPG135001S30, SW36 CPG135001S30, SW37 CPG135001S30, SW38 CPG135001S30, SW39 CPG135001S30, SW4 CPG135001S30, SW40 CPG135001S30, SW41 CPG135001S30, SW42 CPG135001S30, SW43 SK12D07VG4, SW5 CPG135001S30, SW6 CPG135001S30, SW7 CPG135001S30, SW8 CPG135001S30, SW9 CPG135001S30, U1 nice_nano

Commit message: beautify
Changed lines of the file:
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@@
 			(drillshape 0)
 			(scaleselection 1)
-			(outputdirectory "./fab")
+			(outputdirectory "./gerber")
 		)
 	)
@@
 				(type solid)
 			)
-			(layer "B.SilkS")
-		)
-		(fp_line
-			(start 15.24 8.89)
-			(end 15.24 -8.89)
-			(stroke
-				(width 0.381)
-				(type solid)
-			)
-			(layer "B.SilkS")
-		)
-		(fp_line
-			(start -17.78 -8.89)
-			(end -17.78 8.89)
-			(stroke
-				(width 0.381)
-				(type solid)
-			)
-			(layer "B.SilkS")
-		)
-		(fp_line
-			(start 15.24 -8.89)
-			(end -17.78 -8.89)
-			(stroke
-				(width 0.381)
-				(type solid)
-			)
-			(layer "B.SilkS")
-		)
-		(fp_line
-			(start -17.78 8.89)
-			(end -15.24 8.89)
-			(stroke
-				(width 0.381)
-				(type solid)
-			)
-			(layer "F.SilkS")
-		)
-		(fp_line
-			(start -15.24 8.89)
-			(end 15.24 8.89)
-			(stroke
-				(width 0.381)
-				(type solid)
-			)
-			(layer "F.SilkS")
+			(layer "Dwgs.User")
 		)
 		(fp_line
@@
 				(type solid)
 			)
-			(layer "F.SilkS")
-		)
-		(fp_line
-			(start -17.78 -8.89)
-			(end -17.78 8.89)
-			(stroke
-				(width 0.381)
-				(type solid)
-			)
-			(layer "F.SilkS")
-		)
-		(fp_line
-			(start -15.24 -8.89)
-			(end -17.78 -8.89)
-			(stroke
-				(width 0.381)
-				(type solid)
-			)
-			(layer "F.SilkS")
-		)
-		(fp_line
-			(start 15.24 -8.89)
-			(end -15.24 -8.89)
-			(stroke
-				(width 0.381)
-				(type solid)
-			)
-			(layer "F.SilkS")
+			(layer "Dwgs.User")
 		)
 		(fp_line
@@
 			(layer "Dwgs.User")
 		)
+		(fp_line
+			(start -17.78 -8.89)
+			(end -17.78 8.89)
+			(stroke
+				(width 0.381)
+				(type solid)
+			)
+			(layer "Dwgs.User")
+		)
+		(fp_line
+			(start 15.24 -8.89)
+			(end -17.78 -8.89)
+			(stroke
+				(width 0.381)
+				(type solid)
+			)
+			(layer "Dwgs.User")
+		)
 		(fp_text user "GND"
 			(at -11.43 -5.454667 0)
@@
 		)
 		(fp_text user "nice!nano"
-			(at 13.462 -0.254 0)
+			(at -2.6 0 0)
 			(layer "F.SilkS")
 			(effects
 				(font
-					(size 1.5 1.5)
-					(thickness 0.3)
+					(size 1 1)
+					(thickness 0.25)
 				)
 			)
@@
 		(sheetname "Matrix")
 		(sheetfile "sheet_matrix.kicad_sch")
-		(attr smd)
+		(attr smd dnp)
 		(fp_line
 			(start -2.01 -0.85)
@@
 		(sheetname "Matrix")
 		(sheetfile "sheet_matrix.kicad_sch")
-		(attr smd)
+		(attr smd dnp)
 		(fp_line
 			(start -2.01 -0.85)
@@
 		(sheetname "Matrix")
 		(sheetfile "sheet_matrix.kicad_sch")
-		(attr smd)
+		(attr smd dnp)
 		(fp_line
 			(start -2.01 -0.85)
@@
 		(sheetname "Matrix")
 		(sheetfile "sheet_matrix.kicad_sch")
-		(attr smd)
+		(attr smd dnp)
 		(fp_line
 			(start -2.01 -0.85)
@@
 		(sheetname "Matrix")
 		(sheetfile "sheet_matrix.kicad_sch")
-		(attr smd)
+		(attr smd dnp)
 		(fp_line
 			(start -2.01 -0.85)
@@
 		(sheetname "Matrix")
 		(sheetfile "sheet_matrix.kicad_sch")
-		(attr smd)
+		(attr smd dnp)
 		(fp_line
 			(start -2.01 -0.85)
@@
 		(sheetname "Matrix")
 		(sheetfile "sheet_matrix.kicad_sch")
-		(attr smd)
+		(attr smd dnp)
 		(fp_line
 			(start -2.01 -0.85)
@@
 		(sheetname "Matrix")
 		(sheetfile "sheet_matrix.kicad_sch")
-		(attr smd)
+		(attr smd dnp)
 		(fp_line
 			(start -2.01 -0.85)
@@
 		(sheetname "Matrix")
 		(sheetfile "sheet_matrix.kicad_sch")
-		(attr smd)
+		(attr smd dnp)
 		(fp_line
 			(start -2.01 -0.85)
@@
 		(sheetname "Matrix")
 		(sheetfile "sheet_matrix.kicad_sch")
-		(attr smd)
+		(attr smd dnp)
 		(fp_line
 			(start -2.01 -0.85)
@@
 		(sheetname "Matrix")
 		(sheetfile "sheet_matrix.kicad_sch")
-		(attr smd)
+		(attr smd dnp)
 		(fp_line
 			(start -2.01 -0.85)
@@
 		(sheetname "Matrix")
 		(sheetfile "sheet_matrix.kicad_sch")
-		(attr smd)
+		(attr smd dnp)
 		(fp_line
 			(start -2.01 -0.85)
@@
 		(sheetname "Matrix")
 		(sheetfile "sheet_matrix.kicad_sch")
-		(attr smd)
+		(attr smd dnp)
 		(fp_line
 			(start -2.01 -0.85)
@@
 		(sheetname "Matrix")
 		(sheetfile "sheet_matrix.kicad_sch")
-		(attr smd)
+		(attr smd dnp)
 		(fp_line
 			(start -2.01 -0.85)
@@
 		(sheetname "Matrix")
 		(sheetfile "sheet_matrix.kicad_sch")
-		(attr smd)
+		(attr smd dnp)
 		(fp_line
 			(start -2.01 -0.85)
@@
 		(sheetname "Matrix")
 		(sheetfile "sheet_matrix.kicad_sch")
-		(attr smd)
+		(attr smd dnp)
 		(fp_line
 			(start -2.01 -0.85)
@@
 		(sheetname "Matrix")
 		(sheetfile "sheet_matrix.kicad_sch")
-		(attr smd)
+		(attr smd dnp)
 		(fp_line
 			(start -2.01 -0.85)
@@
 		(sheetname "Matrix")
 		(sheetfile "sheet_matrix.kicad_sch")
-		(attr smd)
+		(attr smd dnp)
 		(fp_line
 			(start -2.01 -0.85)
@@
 		(sheetname "Matrix")
 		(sheetfile "sheet_matrix.kicad_sch")
-		(attr smd)
+		(attr smd dnp)
 		(fp_line
 			(start -2.01 -0.85)
@@
 		(sheetname "Matrix")
 		(sheetfile "sheet_matrix.kicad_sch")
-		(attr smd)
+		(attr smd dnp)
 		(fp_line
 			(start -2.01 -0.85)
@@
 		(sheetname "Matrix")
 		(sheetfile "sheet_matrix.kicad_sch")
-		(attr smd)
+		(attr smd dnp)
 		(fp_line
 			(start -2.01 -0.85)
@@
 		)
 		(fp_text user "Battery"
-			(at -3.987088 0 360)
+			(at -3.987088 0 0)
 			(layer "B.SilkS")
 			(effects
@@
 		)
 		(fp_text user "(-)"
-			(at 1.8 2.5 360)
+			(at 1.8 2.5 0)
 			(layer "B.SilkS")
 			(effects
@@
 		)
 		(fp_text user "(+)"
-			(at -1.8 2.5 360)
+			(at -1.8 2.5 0)
 			(layer "B.SilkS")
 			(effects
@@
 		(sheetname "Matrix")
 		(sheetfile "sheet_matrix.kicad_sch")
-		(attr smd)
+		(attr smd dnp)
 		(fp_line
 			(start -2.01 -0.85)
@@
 		(sheetname "Matrix")
 		(sheetfile "sheet_matrix.kicad_sch")
-		(attr smd)
+		(attr smd dnp)
 		(fp_line
 			(start -2.01 -0.85)
@@
 		(sheetname "Matrix")
 		(sheetfile "sheet_matrix.kicad_sch")
-		(attr smd)
+		(attr smd dnp)
 		(fp_line
 			(start -2.01 -0.85)
@@
 		(sheetname "Matrix")
 		(sheetfile "sheet_matrix.kicad_sch")
-		(attr smd)
+		(attr smd dnp)
 		(fp_line
 			(start -2.01 -0.85)
@@
 		(sheetname "Matrix")
 		(sheetfile "sheet_matrix.kicad_sch")
-		(attr smd)
+		(attr smd dnp)
 		(fp_line
 			(start -2.01 -0.85)
@@
 		(sheetname "Matrix")
 		(sheetfile "sheet_matrix.kicad_sch")
-		(attr smd)
+		(attr smd dnp)
 		(fp_line
 			(start -2.01 -0.85)
@@
 		(sheetname "Matrix")
 		(sheetfile "sheet_matrix.kicad_sch")
-		(attr smd)
+		(attr smd dnp)
 		(fp_line
 			(start -2.01 -0.85)
@@
 		(sheetname "Matrix")
 		(sheetfile "sheet_matrix.kicad_sch")
-		(attr smd)
+		(attr smd dnp)
 		(fp_line
 			(start -2.01 -0.85)
@@
 		(sheetname "Matrix")
 		(sheetfile "sheet_matrix.kicad_sch")
-		(attr smd)
+		(attr smd dnp)
 		(fp_line
 			(start -2.01 -0.85)
@@
 		(sheetname "Matrix")
 		(sheetfile "sheet_matrix.kicad_sch")
-		(attr smd)
+		(attr smd dnp)
 		(fp_line
 			(start -2.01 -0.85)
@@
 		(sheetname "Matrix")
 		(sheetfile "sheet_matrix.kicad_sch")
-		(attr smd)
+		(attr smd dnp)
 		(fp_line
 			(start -2.01 -0.85)
@@
 		(sheetname "Matrix")
 		(sheetfile "sheet_matrix.kicad_sch")
-		(attr smd)
+		(attr smd dnp)
 		(fp_line
 			(start -2.01 -0.85)
@@
 		(sheetname "Matrix")
 		(sheetfile "sheet_matrix.kicad_sch")
-		(attr smd)
+		(attr smd dnp)
 		(fp_line
 			(start -2.01 -0.85)
@@
 		(sheetname "Matrix")
 		(sheetfile "sheet_matrix.kicad_sch")
-		(attr smd)
+		(attr smd dnp)
 		(fp_line
 			(start -2.01 -0.85)
@@
 		(sheetname "Matrix")
 		(sheetfile "sheet_matrix.kicad_sch")
-		(attr smd)
+		(attr smd dnp)
 		(fp_line
 			(start -2.01 -0.85)
@@
 		(sheetname "Matrix")
 		(sheetfile "sheet_matrix.kicad_sch")
-		(attr smd)
+		(attr smd dnp)
 		(fp_line
 			(start -2.01 -0.85)
@@
 		(sheetname "Matrix")
 		(sheetfile "sheet_matrix.kicad_sch")
-		(attr smd)
+		(attr smd dnp)
 		(fp_line
 			(start -2.01 -0.85)
@@
 		(sheetname "Matrix")
 		(sheetfile "sheet_matrix.kicad_sch")
-		(attr smd)
+		(attr smd dnp)
 		(fp_line
 			(start -2.01 -0.85)
@@
 		(sheetname "Matrix")
 		(sheetfile "sheet_matrix.kicad_sch")
-		(attr smd)
+		(attr smd dnp)
 		(fp_line
 			(start -2.01 -0.85)
@@
 		(sheetname "Matrix")
 		(sheetfile "sheet_matrix.kicad_sch")
-		(attr smd)
+		(attr smd dnp)
 		(fp_line
 			(start -2.01 -0.85)
@@
 		(sheetname "Matrix")
 		(sheetfile "sheet_matrix.kicad_sch")
-		(attr smd)
+		(attr smd dnp)
 		(fp_line
 			(start -2.01 -0.85)

Commit message: major changes, add plate
Parts:
- removed H_M2_7: MountingHole, MountingHole:MountingHole_2.2mm_M2
- added RST2: SW_Push, itsdmd:SW-T_SPST_TL3342, B.Cu at (148.2, 67.9)
- BATT1: footprint Keyboard:Battery_pads -> itsdmd:Battery_Pads-dual-side; moved to F.Cu
- D1, D10, D11, D12, D13, D14, D15, D16, D17, D18, D19, D2, D20, D21, D22, D23, D24, D25, D26, D27, D28, D29, D3, D30, D31, D32, D33, D34, D35, D36, D37, D38, D39, D4, D40, D41, D42, D5, D6, D7, D8, D9: footprint Diode_SMD:D_SOD-323_HandSoldering -> itsdmd:D_SOD-123
- SW1, SW10, SW11, SW12, SW13, SW14, SW15, SW16, SW17, SW18, SW19, SW2, SW20, SW21, SW22, SW23, SW24, SW25, SW26, SW27, SW28, SW29, SW3, SW30, SW31, SW32, SW33, SW34, SW35, SW36, SW37, SW38, SW39, SW4, SW40, SW41, SW42, SW5, SW6, SW7, SW8, SW9: footprint Keyboard:Kailh_socket_Choc_optional -> itsdmd:KS_Socket_Choc
- SW43: footprint Switch:SK12D07VG4 -> itsdmd:SW-S_SK12D07VG4
- SW_RST1: footprint Switch:KG1 -> itsdmd:SW-S_7.4x2.6-4pad-smd
- U1: footprint ProMicro:nice_nano -> itsdmd:MCB_nice-nano_flip
- moved H_M2_6 96.1 mm to (148.3, 137.7)
- moved H_M2_5 61.7 mm to (239.6, 109.9)
- moved H_M2_4 46.6 mm to (210.1, 55.4)
- moved BATT1 39.5 mm to (135.7, 59.7), turned to 0 degrees
- moved SW43 31.8 mm to (132.4, 55.4), turned to 0 degrees
- moved H_M2_3 30.2 mm to (148.3, 89.3)
- moved SW_RST1 29.6 mm to (161.8, 54.4)
- moved D24 16.7 mm to (189.6, 119.0)
- moved D26 16.7 mm to (194.9, 77.1)
- moved D28 16.7 mm to (205.4, 109.4)
- moved D29 16.7 mm to (210.7, 125.6)
- moved D34 16.7 mm to (229.2, 66.0)
- moved D39 16.7 mm to (258.1, 96.7)
- moved D40 16.7 mm to (266.0, 62.8)
- moved D30 16.7 mm to (210.7, 67.5)
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Connections:
- BATT1 pad 1: RAW -> Net-(BATT1-+)
- BATT1 pad 2: Net-(BATT1--) -> GND
- SW43 pad 2: Net-(BATT1--) -> Net-(BATT1-+)
- SW43 pad COM: GND -> RAW
- SW_RST1 pad 1: RST -> GND
- SW_RST1 pad 2: GND -> RST
- U1 pad 10: COL5 -> COL6
- U1 pad 11: ROW0 -> ROW2
- U1 pad 12: ROW1 -> ROW3
- U1 pad 13: ROW3 -> ROW1
- U1 pad 14: ROW2 -> ROW0
- U1 pad 15: COL6 -> COL5
- U1 pad 16: COL7 -> COL4
- U1 pad 17: COL8 -> COL3
- U1 pad 18: COL9 -> COL2
- U1 pad 19: COL10 -> COL1
- U1 pad 20: COL11 -> COL0
- U1 pad 5: COL0 -> COL11
- U1 pad 6: COL1 -> COL10
- U1 pad 7: COL2 -> COL9
- U1 pad 8: COL3 -> COL8
- U1 pad 9: COL4 -> COL7
Routing:
- net COL3: track 160.5 -> 101.5 mm, vias 3 -> 0
- net COL4: track 126.4 -> 84.1 mm, vias 1 -> 0
- net COL5: track 109.3 -> 68.8 mm, vias 1 -> 0
- net COL1: track 162.9 -> 123.1 mm, vias 3 -> 0
- net COL2: track 144.0 -> 105.0 mm, vias 2 -> 0
- net COL7: track 109.9 -> 77.1 mm, vias 3 -> 0
- net COL9: track 126.5 -> 97.5 mm, vias 3 -> 0
- net COL11: track 160.3 -> 135.3 mm
- net Net-(D31-A): track 31.4 -> 6.71 mm
- net ROW2: track 336.2 -> 311.7 mm, vias 0 -> 1
- net Net-(D27-A): track 30.9 -> 6.71 mm
- net COL8: track 118.5 -> 94.5 mm, vias 2 -> 0
- net COL6: track 87.0 -> 63.2 mm, vias 2 -> 0
- net Net-(D38-A): track 28.3 -> 6.71 mm
- net Net-(D36-A): track 27.8 -> 6.71 mm
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Other:
- board text added: "+ BAT -"
- board text added: "- BAT +"
- board text added: "RST1"
- board text added: "RST2"
- board text removed: "7.0x2.8"
- board text removed: "RST"
- board text removed: "SK12D07"
