File: ozprey_pcb/sheet_matrix.kicad_sch (KiCad schematic)
At the start: 84 parts, among them SW1 CPG135001S30, SW10 CPG135001S30, SW11 CPG135001S30, SW12 CPG135001S30, SW13 CPG135001S30, SW14 CPG135001S30, SW15 CPG135001S30, SW16 CPG135001S30, SW17 CPG135001S30, SW18 CPG135001S30, SW19 CPG135001S30, SW2 CPG135001S30, SW20 CPG135001S30, SW21 CPG135001S30, SW22 CPG135001S30, SW23 CPG135001S30, SW24 CPG135001S30, SW25 CPG135001S30, SW26 CPG135001S30, SW27 CPG135001S30, SW28 CPG135001S30, SW29 CPG135001S30, SW3 CPG135001S30, SW30 CPG135001S30, SW31 CPG135001S30, SW32 CPG135001S30, SW33 CPG135001S30, SW34 CPG135001S30, SW35 CPG135001S30, SW36 CPG135001S30, SW37 CPG135001S30, SW38 CPG135001S30, SW39 CPG135001S30, SW4 CPG135001S30, SW40 CPG135001S30, SW41 CPG135001S30, SW42 CPG135001S30, SW5 CPG135001S30, SW6 CPG135001S30, SW7 CPG135001S30, SW8 CPG135001S30, SW9 CPG135001S30

Commit message: rework pcb, remove enclosure & plate folders
Parts:
- SW1: footprint kapee-keeb-parts:SW_choc_HS_1u -> Keyboard:Kailh_socket_Choc_optional
- SW10: renamed from SW4; footprint kapee-keeb-parts:SW_choc_HS_1u -> Keyboard:Kailh_socket_Choc_optional
- SW11: renamed from SW16; footprint kapee-keeb-parts:SW_choc_HS_1u -> Keyboard:Kailh_socket_Choc_optional
- SW12: renamed from SW28; footprint kapee-keeb-parts:SW_choc_HS_1u -> Keyboard:Kailh_socket_Choc_optional
- SW13: renamed from SW37; footprint kapee-keeb-parts:SW_choc_HS_1u -> Keyboard:Kailh_socket_Choc_optional
- SW14: renamed from SW5; footprint kapee-keeb-parts:SW_choc_HS_1u -> Keyboard:Kailh_socket_Choc_optional
- SW15: renamed from SW17; footprint kapee-keeb-parts:SW_choc_HS_1u -> Keyboard:Kailh_socket_Choc_optional
- SW16: renamed from SW29; footprint kapee-keeb-parts:SW_choc_HS_1u -> Keyboard:Kailh_socket_Choc_optional
- SW17: renamed from SW38; footprint kapee-keeb-parts:SW_choc_HS_1u -> Keyboard:Kailh_socket_Choc_optional
- SW18: renamed from SW6; footprint kapee-keeb-parts:SW_choc_HS_1u -> Keyboard:Kailh_socket_Choc_optional
- SW19: renamed from SW18; footprint kapee-keeb-parts:SW_choc_HS_1u -> Keyboard:Kailh_socket_Choc_optional
- SW2: renamed from SW13; footprint kapee-keeb-parts:SW_choc_HS_1u -> Keyboard:Kailh_socket_Choc_optional
- SW20: renamed from SW30; footprint kapee-keeb-parts:SW_choc_HS_1u -> Keyboard:Kailh_socket_Choc_optional
- SW21: renamed from SW39; footprint kapee-keeb-parts:SW_choc_HS_1.5u -> Keyboard:Kailh_socket_Choc_optional
- SW22: renamed from SW7; footprint kapee-keeb-parts:SW_choc_HS_1u -> Keyboard:Kailh_socket_Choc_optional
- SW23: renamed from SW19; footprint kapee-keeb-parts:SW_choc_HS_1u -> Keyboard:Kailh_socket_Choc_optional
- SW24: renamed from SW31; footprint kapee-keeb-parts:SW_choc_HS_1u -> Keyboard:Kailh_socket_Choc_optional
- SW25: renamed from SW40; footprint kapee-keeb-parts:SW_choc_HS_1.5u -> Keyboard:Kailh_socket_Choc_optional
- SW26: renamed from SW8; footprint kapee-keeb-parts:SW_choc_HS_1u -> Keyboard:Kailh_socket_Choc_optional
- SW27: renamed from SW20; footprint kapee-keeb-parts:SW_choc_HS_1u -> Keyboard:Kailh_socket_Choc_optional
- SW28: renamed from SW32; footprint kapee-keeb-parts:SW_choc_HS_1u -> Keyboard:Kailh_socket_Choc_optional
- SW29: renamed from SW41; footprint kapee-keeb-parts:SW_choc_HS_1u -> Keyboard:Kailh_socket_Choc_optional
- SW3: renamed from SW25; footprint kapee-keeb-parts:SW_choc_HS_1u -> Keyboard:Kailh_socket_Choc_optional
- SW30: renamed from SW9; footprint kapee-keeb-parts:SW_choc_HS_1u -> Keyboard:Kailh_socket_Choc_optional
- SW31: renamed from SW21; footprint kapee-keeb-parts:SW_choc_HS_1u -> Keyboard:Kailh_socket_Choc_optional
- SW32: renamed from SW33; footprint kapee-keeb-parts:SW_choc_HS_1u -> Keyboard:Kailh_socket_Choc_optional
- SW33: renamed from SW42; footprint kapee-keeb-parts:SW_choc_HS_1u -> Keyboard:Kailh_socket_Choc_optional
- SW34: renamed from SW10; footprint kapee-keeb-parts:SW_choc_HS_1u -> Keyboard:Kailh_socket_Choc_optional
- SW35: renamed from SW22; footprint kapee-keeb-parts:SW_choc_HS_1u -> Keyboard:Kailh_socket_Choc_optional
- SW36: renamed from SW34; footprint kapee-keeb-parts:SW_choc_HS_1u -> Keyboard:Kailh_socket_Choc_optional
- SW37: renamed from SW11; footprint kapee-keeb-parts:SW_choc_HS_1u -> Keyboard:Kailh_socket_Choc_optional
- SW38: renamed from SW23; footprint kapee-keeb-parts:SW_choc_HS_1u -> Keyboard:Kailh_socket_Choc_optional
- SW39: renamed from SW35; footprint kapee-keeb-parts:SW_choc_HS_1u -> Keyboard:Kailh_socket_Choc_optional
- SW4: renamed from SW2; footprint kapee-keeb-parts:SW_choc_HS_1u -> Keyboard:Kailh_socket_Choc_optional
- SW40: renamed from SW12; footprint kapee-keeb-parts:SW_choc_HS_1u -> Keyboard:Kailh_socket_Choc_optional
- SW41: renamed from SW24; footprint kapee-keeb-parts:SW_choc_HS_1u -> Keyboard:Kailh_socket_Choc_optional
- SW42: renamed from SW36; footprint kapee-keeb-parts:SW_choc_HS_1u -> Keyboard:Kailh_socket_Choc_optional
- SW5: renamed from SW14; footprint kapee-keeb-parts:SW_choc_HS_1u -> Keyboard:Kailh_socket_Choc_optional
- SW6: renamed from SW26; footprint kapee-keeb-parts:SW_choc_HS_1u -> Keyboard:Kailh_socket_Choc_optional
- SW7: renamed from SW3; footprint kapee-keeb-parts:SW_choc_HS_1u -> Keyboard:Kailh_socket_Choc_optional
- SW8: renamed from SW15; footprint kapee-keeb-parts:SW_choc_HS_1u -> Keyboard:Kailh_socket_Choc_optional
- SW9: renamed from SW27; footprint kapee-keeb-parts:SW_choc_HS_1u -> Keyboard:Kailh_socket_Choc_optional
- renumbered D4 to D10, D16 to D11, D28 to D12, D37 to D13, D5 to D14, D17 to D15, D29 to D16, D38 to D17, D6 to D18, D18 to D19, D13 to D2, D30 to D20, D39 to D21, D7 to D22, D19 to D23, D31 to D24, D40 to D25, D8 to D26, D20 to D27, D32 to D28, D41 to D29, D25 to D3, D9 to D30, D21 to D31, D33 to D32, D42 to D33, D10 to D34, D22 to D35, D34 to D36, D11 to D37, D23 to D38, D35 to D39, D2 to D4, D12 to D40, D24 to D41, D36 to D42, D14 to D5, D26 to D6, D3 to D7, D15 to D8, D27 to D9
Other:
- company: (none) -> itsdmd
- title: (none) -> Matrix

Commit message: beautify
Parts:
- D1, D10, D11, D12, D13, D14, D15, D16, D17, D18, D19, D2, D20, D21, D22, D23, D24, D25, D26, D27, D28, D29, D3, D30, D31, D32, D33, D34, D35, D36, D37, D38, D39, D4, D40, D41, D42, D5, D6, D7, D8, D9: now not fitted
Changed lines of the file:
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@@
 		(in_bom yes)
 		(on_board yes)
-		(dnp no)
+		(dnp yes)
 		(fields_autoplaced yes)
 		(property "Reference" "D21"
@@
 		(in_bom yes)
 		(on_board yes)
-		(dnp no)
+		(dnp yes)
 		(fields_autoplaced yes)
 		(property "Reference" "D22"
@@
 		(in_bom yes)
 		(on_board yes)
-		(dnp no)
+		(dnp yes)
 		(fields_autoplaced yes)
 		(property "Reference" "D26"
@@
 		(in_bom yes)
 		(on_board yes)
-		(dnp no)
+		(dnp yes)
 		(fields_autoplaced yes)
 		(property "Reference" "D17"
@@
 		(in_bom yes)
 		(on_board yes)
-		(dnp no)
+		(dnp yes)
 		(fields_autoplaced yes)
 		(property "Reference" "D42"
@@
 		(in_bom yes)
 		(on_board yes)
-		(dnp no)
+		(dnp yes)
 		(fields_autoplaced yes)
 		(property "Reference" "D34"
@@
 		(in_bom yes)
 		(on_board yes)
-		(dnp no)
+		(dnp yes)
 		(fields_autoplaced yes)
 		(property "Reference" "D14"
@@
 		(in_bom yes)
 		(on_board yes)
-		(dnp no)
+		(dnp yes)
 		(fields_autoplaced yes)
 		(property "Reference" "D30"
@@
 		(in_bom yes)
 		(on_board yes)
-		(dnp no)
+		(dnp yes)
 		(fields_autoplaced yes)
 		(property "Reference" "D9"
@@
 		(in_bom yes)
 		(on_board yes)
-		(dnp no)
+		(dnp yes)
 		(fields_autoplaced yes)
 		(property "Reference" "D15"
@@
 		(in_bom yes)
 		(on_board yes)
-		(dnp no)
+		(dnp yes)
 		(fields_autoplaced yes)
 		(property "Reference" "D3"
@@
 		(in_bom yes)
 		(on_board yes)
-		(dnp no)
+		(dnp yes)
 		(fields_autoplaced yes)
 		(property "Reference" "D27"
@@
 		(in_bom yes)
 		(on_board yes)
-		(dnp no)
+		(dnp yes)
 		(fields_autoplaced yes)
 		(property "Reference" "D1"
@@
 		(in_bom yes)
 		(on_board yes)
-		(dnp no)
+		(dnp yes)
 		(fields_autoplaced yes)
 		(property "Reference" "D6"
@@
 		(in_bom yes)
 		(on_board yes)
-		(dnp no)
+		(dnp yes)
 		(fields_autoplaced yes)
 		(property "Reference" "D20"
@@
 		(in_bom yes)
 		(on_board yes)
-		(dnp no)
+		(dnp yes)
 		(fields_autoplaced yes)
 		(property "Reference" "D19"
@@
 		(in_bom yes)
 		(on_board yes)
-		(dnp no)
+		(dnp yes)
 		(fields_autoplaced yes)
 		(property "Reference" "D5"
@@
 		(in_bom yes)
 		(on_board yes)
-		(dnp no)
+		(dnp yes)
 		(fields_autoplaced yes)
 		(property "Reference" "D18"
@@
 		(in_bom yes)
 		(on_board yes)
-		(dnp no)
+		(dnp yes)
 		(fields_autoplaced yes)
 		(property "Reference" "D31"
@@
 		(in_bom yes)
 		(on_board yes)
-		(dnp no)
+		(dnp yes)
 		(fields_autoplaced yes)
 		(property "Reference" "D10"
@@
 		(in_bom yes)
 		(on_board yes)
-		(dnp no)
+		(dnp yes)
 		(fields_autoplaced yes)
 		(property "Reference" "D32"
@@
 		(in_bom yes)
 		(on_board yes)
-		(dnp no)
+		(dnp yes)
 		(fields_autoplaced yes)
 		(property "Reference" "D7"
@@
 		(in_bom yes)
 		(on_board yes)
-		(dnp no)
+		(dnp yes)
 		(property "Reference" "D39"
 			(at 228.6 92.7099 90)
@@
 		(in_bom yes)
 		(on_board yes)
-		(dnp no)
+		(dnp yes)
 		(fields_autoplaced yes)
 		(property "Reference" "D8"
@@
 		(in_bom yes)
 		(on_board yes)
-		(dnp no)
+		(dnp yes)
 		(property "Reference" "D38"
 			(at 228.6 71.7549 90)
@@
 		(in_bom yes)
 		(on_board yes)
-		(dnp no)
+		(dnp yes)
 		(property "Reference" "D12"
 			(at 81.28 92.7099 90)
@@
 		(in_bom yes)
 		(on_board yes)
-		(dnp no)
+		(dnp yes)
 		(property "Reference" "D13"
 			(at 81.28 110.4899 90)
@@
 		(in_bom yes)
 		(on_board yes)
-		(dnp no)
+		(dnp yes)
 		(fields_autoplaced yes)
 		(property "Reference" "D11"
@@
 		(in_bom yes)
 		(on_board yes)
-		(dnp no)
+		(dnp yes)
 		(fields_autoplaced yes)
 		(property "Reference" "D4"
@@
 		(in_bom yes)
 		(on_board yes)
-		(dnp no)
+		(dnp yes)
 		(fields_autoplaced yes)
 		(property "Reference" "D36"
@@
 		(in_bom yes)
 		(on_board yes)
-		(dnp no)
+		(dnp yes)
 		(fields_autoplaced yes)
 		(property "Reference" "D35"
@@
 		(in_bom yes)
 		(on_board yes)
-		(dnp no)
+		(dnp yes)
 		(fields_autoplaced yes)
 		(property "Reference" "D24"
@@
 		(in_bom yes)
 		(on_board yes)
-		(dnp no)
+		(dnp yes)
 		(fields_autoplaced yes)
 		(property "Reference" "D28"
@@
 		(in_bom yes)
 		(on_board yes)
-		(dnp no)
+		(dnp yes)
 		(fields_autoplaced yes)
 		(property "Reference" "D25"
@@
 		(in_bom yes)
 		(on_board yes)
-		(dnp no)
+		(dnp yes)
 		(property "Reference" "D2"
 			(at 26.67 71.7549 90)
@@
 		(in_bom yes)
 		(on_board yes)
-		(dnp no)
+		(dnp yes)
 		(fields_autoplaced yes)
 		(property "Reference" "D33"
@@
 		(in_bom yes)
 		(on_board yes)
-		(dnp no)
+		(dnp yes)
 		(fields_autoplaced yes)
 		(property "Reference" "D40"
@@
 		(in_bom yes)
 		(on_board yes)
-		(dnp no)
+		(dnp yes)
 		(property "Reference" "D37"
 			(at 228.6 49.5299 90)
@@
 		(in_bom yes)
 		(on_board yes)
-		(dnp no)
+		(dnp yes)
 		(fields_autoplaced yes)
 		(property "Reference" "D23"
@@
 		(in_bom yes)
 		(on_board yes)
-		(dnp no)
+		(dnp yes)
 		(fields_autoplaced yes)
 		(property "Reference" "D41"
@@
 		(in_bom yes)
 		(on_board yes)
-		(dnp no)
+		(dnp yes)
 		(fields_autoplaced yes)
 		(property "Reference" "D29"
@@
 		(in_bom yes)
 		(on_board yes)
-		(dnp no)
+		(dnp yes)
 		(property "Reference" "D16"
 			(at 99.06 92.7099 90)

Commit message: major changes, add plate
Parts:
- D1, D10, D11, D12, D13, D14, D15, D16, D17, D18, D19, D2, D20, D21, D22, D23, D24, D25, D26, D27, D28, D29, D3, D30, D31, D32, D33, D34, D35, D36, D37, D38, D39, D4, D40, D41, D42, D5, D6, D7, D8, D9: footprint Diode_SMD:D_SOD-323_HandSoldering -> itsdmd:D_SOD-123
- SW1, SW10, SW11, SW12, SW13, SW14, SW15, SW16, SW17, SW18, SW19, SW2, SW20, SW21, SW22, SW23, SW24, SW25, SW26, SW27, SW28, SW29, SW3, SW30, SW31, SW32, SW33, SW34, SW35, SW36, SW37, SW38, SW39, SW4, SW40, SW41, SW42, SW5, SW6, SW7, SW8, SW9: footprint Keyboard:Kailh_socket_Choc_optional -> itsdmd:KS_Socket_Choc
